File: FRDM-SX1255.kicad_sch (KiCad schematic)
At the start: 72 parts, among them IC1 SX1255, J5 RX, J6 TX, J7 D_I2C OLED, Q1 BSS84, U1 MCP1703Ax-330xxDB, X1 B3909, Y1 38.4MHz

Commit message: Add files via upload
Parts:
- L2: Manufacturer Johanson Technology Inc. -> Murata Electronics; Manufacturer Product Number LRC0603CJ82NGV001T -> LQW18AS82NG00D; Part Number 712-LRC0603CJ82NGV001TCT-ND -> 490-LQW18AS82NG00DCT-ND
- L3: Manufacturer Johanson Technology Inc. -> Murata Electronics; Manufacturer Product Number LRC0603CJ39NGV001T -> LQW18AS39NG00D; Part Number 712-LRC0603CJ39NGV001TCT-ND -> 490-LQW18AS39NG00DCT-ND
Changed lines of the file:
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@@
 	(title_block
 		(title "FRDM-MCXN947 + SX1255")
-		(date "2026-10-28")
+		(date "2026-10-29")
 		(rev "V1.3")
 		(company "Z32IT, DM5LF")
@@
 			)
 		)
-		(property "Manufacturer" "Johanson Technology Inc."
+		(property "Manufacturer" "Murata Electronics"
 			(at 213.36 55.88 0)
 			(hide yes)
@@
 			)
 		)
-		(property "Manufacturer Product Number" "LRC0603CJ82NGV001T"
+		(property "Manufacturer Product Number" "LQW18AS82NG00D"
 			(at 213.36 55.88 0)
 			(hide yes)
@@
 			)
 		)
-		(property "Part Number" "712-LRC0603CJ82NGV001TCT-ND"
+		(property "Part Number" "490-LQW18AS82NG00DCT-ND"
 			(at 213.36 55.88 0)
 			(hide yes)
@@
 			)
 		)
-		(property "Manufacturer" "Johanson Technology Inc."
+		(property "Manufacturer" "Murata Electronics"
 			(at 218.44 50.8 90)
 			(hide yes)
@@
 			)
 		)
-		(property "Manufacturer Product Number" "LRC0603CJ39NGV001T"
+		(property "Manufacturer Product Number" "LQW18AS39NG00D"
 			(at 218.44 50.8 90)
 			(hide yes)
@@
 			)
 		)
-		(property "Part Number" "712-LRC0603CJ39NGV001TCT-ND"
+		(property "Part Number" "490-LQW18AS39NG00DCT-ND"
 			(at 218.44 50.8 90)
 			(hide yes)
