File: FRDM-SX1255.kicad_pcb (KiCad board)
At the start: 2 copper layers, 118 x 55 mm, 78 parts, among them IC1 SX1255, J1 SSQ-108-03-T-D, J12 SSQ-114-03-T-D, J2 SSQ-110-03-T-D, J3 SSQ-108-03-T-D, J4 SSQ-106-03-T-D, J5 RX, J6 TX, J7 D_I2C OLED, J9 SSQ-116-03-T-D, Q1 BSS84, U1 MCP1703Ax-330xxDB, X1 B3909, Y1 38.4MHz

Commit message: Add files via upload
Parts:
- renumbered bypass to JP2
Routing:
- net GND: vias 321 -> 329
Changed lines of the file:
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@@
 	(title_block
 		(title "FRDM-MCXN947 + SX1255")
-		(date "2026-10-28")
+		(date "2026-10-29")
 		(rev "V1.4")
 		(company "Z32IT, DM5LF")
@@
 			)
 		)
-		(property "Manufacturer" "Johanson Technology Inc."
+		(property "Manufacturer" "Murata Electronics"
 			(at 0 0 90)
 			(unlocked yes)
@@
 			)
 		)
-		(property "Manufacturer Product Number" "LRC0603CJ82NGV001T"
+		(property "Manufacturer Product Number" "LQW18AS82NG00D"
 			(at 0 0 90)
 			(unlocked yes)
@@
 			)
 		)
-		(property "Part Number" "712-LRC0603CJ82NGV001TCT-ND"
+		(property "Part Number" "490-LQW18AS82NG00DCT-ND"
 			(at 0 0 90)
 			(unlocked yes)
@@
 		(descr "SMD Solder Jumper, 1x1.5mm, rounded Pads, 0.3mm gap, open")
 		(tags "solder jumper open")
-		(property "Reference" "bypass"
+		(property "Reference" "JP2"
 			(at 0 2 0)
 			(layer "F.SilkS")
@@
 			)
 		)
-		(property "Manufacturer" "Johanson Technology Inc."
+		(property "Manufacturer" "Murata Electronics"
 			(at 0 0 90)
 			(unlocked yes)
@@
 			)
 		)
-		(property "Manufacturer Product Number" "LRC0603CJ39NGV001T"
+		(property "Manufacturer Product Number" "LQW18AS39NG00D"
 			(at 0 0 90)
 			(unlocked yes)
@@
 			)
 		)
-		(property "Part Number" "712-LRC0603CJ39NGV001TCT-ND"
+		(property "Part Number" "490-LQW18AS39NG00DCT-ND"
 			(at 0 0 90)
 			(unlocked yes)
@@
 	)
 	(via
+		(at 84.25 64.5)
+		(size 0.6)
+		(drill 0.3)
+		(layers "F.Cu" "B.Cu")
+		(free yes)
+		(net "GND")
+	)
+	(via
 		(at 138.75 104.5)
 		(size 0.6)
@@
 	)
 	(via
+		(at 84 109.5)
+		(size 0.6)
+		(drill 0.3)
+		(layers "F.Cu" "B.Cu")
+		(free yes)
+		(net "GND")
+	)
+	(via
 		(at 153.5 90.5)
 		(size 0.6)
@@
 	)
 	(via
+		(at 157.75 83.5)
+		(size 0.6)
+		(drill 0.3)
+		(layers "F.Cu" "B.Cu")
+		(free yes)
+		(net "GND")
+	)
+	(via
 		(at 181.907395 93.576366)
 		(size 0.6)
@@
 	)
 	(via
+		(at 84 108.25)
+		(size 0.6)
+		(drill 0.3)
+		(layers "F.Cu" "B.Cu")
+		(free yes)
+		(net "GND")
+	)
+	(via
 		(at 137.75 91.5)
 		(size 0.6)
@@
 	)
 	(via
+		(at 157.75 84)
+		(size 0.6)
+		(drill 0.3)
+		(layers "F.Cu" "B.Cu")
+		(free yes)
+		(net "GND")
+	)
+	(via
 		(at 186.75 98.25)
 		(size 0.6)
@@
 	)
 	(via
+		(at 84.25 65.75)
+		(size 0.6)
+		(drill 0.3)
+		(layers "F.Cu" "B.Cu")
+		(free yes)
+		(net "GND")
+	)
+	(via
 		(at 141.817052 100.685287)
 		(size 0.6)
@@
 	)
 	(via
+		(at 84.25 67)
+		(size 0.6)
+		(drill 0.3)
+		(layers "F.Cu" "B.Cu")
+		(free yes)
+		(net "GND")
+	)
+	(via
 		(at 102.403629 95.501811)
 		(size 0.6)
@@
 		(size 0.6)
 		(drill 0.3)
+		(layers "F.Cu" "B.Cu")
+		(free yes)
+		(net "GND")
+	)
+	(via
+		(at 84 110.75)
+		(size 0.6)
+		(drill 0.3)
