File: FRDM-SX1255+/FRDM-SX1255+.kicad_pcb (KiCad board)
At the start: 2 copper layers, 118 x 55 mm, 86 parts, among them IC1 SX1255, J1 SSQ-108-03-T-D, J12 SSQ-114-03-T-D, J2 SSQ-110-03-T-D, J3 SSQ-108-03-T-D, J4 SSQ-106-03-T-D, J5 RX, J6 TX, J7 D_I2C OLED, J9 SSQ-116-03-T-D, Q1 BSS84, U1 MCP1703Ax-330xxDB, U1 TQP3M9036, X1 B3909, Y1 38.4MHz

Commit message: Add files via upload
Routing:
- net +5V0: track 110.1 -> 111.5 mm, vias 2 -> 1

Commit message: Add files via upload
Routing:
- net GND: vias 490 -> 498
Changed lines of the file:
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@@
+	)
+	(via
+		(at 84.5 66.5)
+		(size 0.6)
+		(drill 0.3)
+		(layers "F.Cu" "B.Cu")
+		(free yes)
+		(net "GND")
 	)
 	(via
@@
 	)
 	(via
+		(at 157.75 84)
+		(size 0.6)
+		(drill 0.3)
+		(layers "F.Cu" "B.Cu")
+		(free yes)
+		(net "GND")
+	)
+	(via
 		(at 172 103.75)
 		(size 0.6)
@@
 	)
 	(via
+		(at 157.75 83.5)
+		(size 0.6)
+		(drill 0.3)
+		(layers "F.Cu" "B.Cu")
+		(free yes)
+		(net "GND")
+	)
+	(via
 		(at 139.5 90.75)
 		(size 0.6)
@@
 	)
 	(via
+		(at 84.5 108)
+		(size 0.6)
+		(drill 0.3)
+		(layers "F.Cu" "B.Cu")
+		(free yes)
+		(net "GND")
+	)
+	(via
 		(at 143.25 104.5)
 		(size 0.6)
@@
 	)
 	(via
+		(at 84.5 67.75)
+		(size 0.6)
+		(drill 0.3)
+		(layers "F.Cu" "B.Cu")
+		(free yes)
+		(net "GND")
+	)
+	(via
 		(at 144.75 109.25)
 		(size 0.6)
@@
 	)
 	(via
+		(at 84.5 65.25)
+		(size 0.6)
+		(drill 0.3)
+		(layers "F.Cu" "B.Cu")
+		(free yes)
+		(net "GND")
+	)
+	(via
 		(at 144.75 100.75)
 		(size 0.6)
@@
 	)
 	(via
+		(at 84.5 109.25)
+		(size 0.6)
+		(drill 0.3)
+		(layers "F.Cu" "B.Cu")
+		(free yes)
+		(net "GND")
+	)
+	(via
 		(at 153.5 103.75)
 		(size 0.6)
@@
 		(size 0.6)
 		(drill 0.3)
+		(layers "F.Cu" "B.Cu")
+		(free yes)
+		(net "GND")
+	)
+	(via
+		(at 84.5 110.5)
+		(size 0.6)
+		(drill 0.3)
